Commit message: 增加 OpenCV程序和lakibeam驱动

File: src/ros_uart_protocol/urdf/nailong_model.urdf (robot description, URDF)
Before this commit: robot mycar, 7 links, 6 joints
Joints:
- removed joint left_wheel2base_link
- removed joint right_wheel2base_link
- added joint wheel_left_joint: type continuous, parent base_link, child left_wheel, origin xyz=0 0.24 -0.0755, axis 0 1 0
- added joint wheel_right_joint: type continuous, parent base_link, child right_wheel, origin xyz=0 -0.24 -0.0755, axis 0 1 0
- joint back_wheel2base_link: type continuous -> fixed
- joint front_wheel2base_link: type continuous -> fixed
